File: zeropi.sch (EAGLE design)
At the start: 1 part, among them U1 STM32F10XRXT6

Commit message: update schematic.
Parts:
- added C10, C11, C12, C13, C5, C6, C7, C8, C9: 100nF, cap-master:CNP-0805
- added C14, C15: 47u, cap-master:CP-153CLV-1012
- added U$1: TLV1117, stm32_usbserial:TLV1117
- added X1: MINI-USB-SCHIELD-32005-301, con-cypressindustries:MINI-USB-SCHIELD-32005-301
Connections:
- new net +3V3: C10.2, C11.2, C12.2, C13.2, C14.+, C5.2, C6.2, C7.2, C8.2, C9.2, U$1.VOUT, U$1.VOUT2
- new net +5V: C15.+, U$1.VIN, X1G$1.1
- new net D+: X1G$1.3
- new net D-: X1G$1.2
- new net GND: C10.1, C11.1, C12.1, C13.1, C14.-, C15.-, C5.1, C6.1, C7.1, C8.1, C9.1, U$1.GND, X1G$1.5, X1S.S1, X1S.S2, X1S.S3, X1S.S4
